File: jumper_pak.kicad_pcb (KiCad board)
At the start: 2 copper layers, 43 x 25 mm, 23 parts, among them J1 n64_exp

Commit message: added README.md
Other:
- net class Default removed

Commit message: added license
Other:
- board text added: "github.com/tehKaiN/jumper_pak"
- board text removed: "github.com/teh_KaiN/jumper_pak"
Changed lines of the file:
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@@
   (gr_line (start 108.9 107.5) (end 108.9 96.7) (layer "Edge.Cuts") (width 0.05))
   (gr_line (start 108.9 107.5) (end 135.4 107.5) (layer "Edge.Cuts") (width 0.05))
-  (gr_text "github.com/teh_KaiN/jumper_pak" (at 122.76 84.02) (layer "B.SilkS")
+  (gr_text "github.com/tehKaiN/jumper_pak" (at 122.76 84.02) (layer "B.SilkS")
     (effects (font (size 1 0.8) (thickness 0.12)) (justify mirror))
   )
